Commit message: files modified

File: robot/urdf/robot.xacro (robot description, xacro)
@@ -31,3 +31,35 @@
     </visual>
   </link>
+  <link name='left_wheel'>
+    <pose>0 0 0 0 0 0</pose>
+    <inertial>
+      <mass value="5.0"/>
+      <origin xyz="0 0 0" rpy="0 0 0"/>
+      <inertia
+          ixx="0.1" ixy="0" ixz="0"
+          iyy="0.1" iyz="0"
+          izz="0.1"
+      />
+    </inertial>
+    <collision name='left_wheel_collision'>
+      <origin xyz="0 0 0" rpy="0 0 0"/>
+      <geometry>
+        <cylinder radius="0.05" length="0.015"/>
+      </geometry>
+    </collision>
+    <visual name='left_wheel_visual'>
+      <origin xyz="0 0 0" rpy="0 0 0"/>
+      <geometry>
+        <cylinder radius="0.05" length="0.015"/>
+      </geometry>
+    </visual>
+  </link>
+  <joint type="continuous" name="left_wheel_hinge">
+    <origin xyz="-0.107266 -0.242145 0.067711" rpy=" 0 -1.5707 -0.001871"/>
+    <child link="left_wheel"/>
+    <parent link="robot_body"/>
+    <axis xyz="0 0 1" rpy="0 0 0"/>
+    <limit effort="10000" velocity="1000"/>
+    <dynamics damping="1.0" friction="1.0"/>
+  </joint>
 </robot>

Commit message: urdf updated

File: robot/urdf/robot.xacro (robot description, xacro)
@@ -11,5 +11,5 @@
     <inertial>
       <mass value="1e-5"/>
-      <origin xyz="0 0 0" rpy=" 0 0 0"/>
+      <origin xyz="0 0 0" rpy=" 1.5707 0 1.5707"/>
       <inertia
           ixx="1e-6" ixy="0" ixz="0"
@@ -19,5 +19,5 @@
     </inertial>
     <collision name='robot_collision'>
-      <origin xyz="0 0 0" rpy=" 0 0 0"/>
+      <origin xyz="0 0 0" rpy=" 1.5707 0 1.5707"/>
       <geometry>
         <box size="0.1 0.1 0.1"/>
@@ -25,5 +25,5 @@
     </collision>
     <visual name='robot_visual'>
-      <origin xyz="0 0 0" rpy=" 0 0 0"/>
+      <origin xyz="0 0 0" rpy=" 1.5707 0 1.5707"/>
       <geometry>
         <mesh filename="package://robot/meshes/Dingo_without_tyre.dae"/>
@@ -56,5 +56,5 @@
   </link>
   <joint type="continuous" name="left_wheel_hinge">
-    <origin xyz="-0.107266 -0.242145 0.067711" rpy=" 0 -1.5707 -0.001871"/>
+    <origin xyz="-0.107266 -0.242145 0.5" rpy=" 0 -1.5707 -0.001871"/>
     <child link="left_wheel"/>
     <parent link="robot_body"/>

Commit message: xacro file updated

File: robot/urdf/robot.xacro (robot description, xacro)
@@ -11,5 +11,5 @@
     <inertial>
       <mass value="1e-5"/>
-      <origin xyz="0 0 0" rpy=" 1.5707 0 1.5707"/>
+      <origin xyz="0 0 0.5" rpy=" 1.5707 0 1.5707"/>
       <inertia
           ixx="1e-6" ixy="0" ixz="0"
@@ -19,5 +19,5 @@
     </inertial>
     <collision name='robot_collision'>
-      <origin xyz="0 0 0" rpy=" 1.5707 0 1.5707"/>
+      <origin xyz="0 0 0.5" rpy=" 1.5707 0 1.5707"/>
       <geometry>
         <box size="0.1 0.1 0.1"/>
@@ -25,5 +25,5 @@
     </collision>
     <visual name='robot_visual'>
-      <origin xyz="0 0 0" rpy=" 1.5707 0 1.5707"/>
+      <origin xyz="0 0 0.5" rpy=" 1.5707 0 1.5707"/>
       <geometry>
         <mesh filename="package://robot/meshes/Dingo_without_tyre.dae"/>
@@ -55,6 +55,30 @@
     </visual>
   </link>
+  <link name='right_wheel'>
+    <pose>0 0 0 0 0 0</pose>
+    <inertial>
+      <mass value="5"/>
+      <origin xyz="0 0 0" rpy="0 0 0"/>
+      <inertia
+          ixx="0.1" ixy="0" ixz="0"
+          iyy="0.1" iyz="0"
+          izz="0.1"
+      />
+    </inertial>
+    <collision name='right_wheel_collision'>
+      <origin xyz="0 0 0" rpy="0 0 0"/>
+      <geometry>
+        <cylinder radius="0.05" length="0.015"/>
+      </geometry>
+    </collision>
+    <visual name='right_wheel_visual'>
+      <origin xyz="0 0 0" rpy="0 0 0"/>
+      <geometry>
+        <cylinder radius="0.05" length="0.015"/>
+      </geometry>
+    </visual>
+  </link>
   <joint type="continuous" name="left_wheel_hinge">
-    <origin xyz="-0.107266 -0.242145 0.5" rpy=" 0 -1.5707 -0.001871"/>
+    <origin xyz="-0.107266 -0.242145 0.5" rpy=" 0 -1.5707 1.5707"/>
     <child link="left_wheel"/>
     <parent link="robot_body"/>
@@ -63,3 +87,11 @@
     <dynamics damping="1.0" friction="1.0"/>
   </joint>
+  <joint type="continuous" name="right_wheel_hinge">
+    <origin xyz="-0.107266 0.242145 0.5" rpy=" 0 -1.5707 1.5707"/>
+    <child link="right_wheel"/>
+    <parent link="robot_body"/>
+    <axis xyz="0 0 1" rpy="0 0 0"/>
+    <limit effort="10000" velocity="1000"/>
+    <dynamics damping="1.0" friction="1.0"/>
+  </joint>
 </robot>

Commit message: values changed in urdf

File: robot/urdf/robot.xacro (robot description, xacro)
@@ -10,5 +10,5 @@
     <pose>0 0 0 0 0 0</pose>
     <inertial>
-      <mass value="1e-5"/>
+      <mass value="8e-5"/>
       <origin xyz="0 0 0.5" rpy=" 1.5707 0 1.5707"/>
       <inertia
@@ -34,5 +34,5 @@
     <pose>0 0 0 0 0 0</pose>
     <inertial>
-      <mass value="5.0"/>
+      <mass value="8.0"/>
       <origin xyz="0 0 0" rpy="0 0 0"/>
       <inertia
@@ -58,5 +58,5 @@
     <pose>0 0 0 0 0 0</pose>
     <inertial>
-      <mass value="5"/>
+      <mass value="8"/>
       <origin xyz="0 0 0" rpy="0 0 0"/>
       <inertia

Commit message: camera_pillar added

File: robot/urdf/robot.xacro (robot description, xacro)
@@ -10,5 +10,5 @@
     <pose>0 0 0 0 0 0</pose>
     <inertial>
-      <mass value="8e-5"/>
+      <mass value="5e-5"/>
       <origin xyz="0 0 0.5" rpy=" 1.5707 0 1.5707"/>
       <inertia
@@ -79,4 +79,28 @@
     </visual>
   </link>
+  <link name='camera_pillar'>
+    <pose>0 0 0 0 0 0</pose>
+    <inertial>
+      <mass value="0.2"/>
+      <origin xyz="0 0 0" rpy="0 0 0"/>
+      <inertia
+          ixx="0.1" ixy="0" ixz="0"
+          iyy="0.1" iyz="0"
+          izz="0.1"
+      />
+    </inertial>
+    <collision name='pillar_collision'>
+      <origin xyz="0 0 0" rpy="0 0 0"/>
+      <geometry>
+        <box size="0.05 0.05 0.2"/>
+      </geometry>
+    </collision>
+    <visual name='pillar_visual'>
+      <origin xyz="0 0 0" rpy="0 0 0"/>
+      <geometry>
+        <box size="0.05 0.05 0.2"/>
+      </geometry>
+    </visual>
+  </link>
   <joint type="continuous" name="left_wheel_hinge">
     <origin xyz="-0.107266 -0.242145 0.5" rpy=" 0 -1.5707 1.5707"/>
@@ -95,3 +119,11 @@
     <dynamics damping="1.0" friction="1.0"/>
   </joint>
+  <joint type="fixed" name="camera_pillar_hinge">
+    <origin xyz="-0.182538 0.002574 0.674205" rpy="-0.000428 0.002653 -0.024756"/>
+    <child link="camera_pillar"/>
+    <parent link="robot_body"/>
+    <axis xyz="0 0 1" rpy="0 0 0"/>
+    <limit effort="10000" velocity="1000"/>
+    <dynamics damping="1.0" friction="1.0"/>
+  </joint>
 </robot>

Commit message: urdf updated

File: robot/urdf/robot.xacro (robot description, xacro)
@@ -10,5 +10,5 @@
     <pose>0 0 0 0 0 0</pose>
     <inertial>
-      <mass value="5e-5"/>
+      <mass value="9"/>
       <origin xyz="0 0 0.5" rpy=" 1.5707 0 1.5707"/>
       <inertia
@@ -34,5 +34,5 @@
     <pose>0 0 0 0 0 0</pose>
     <inertial>
-      <mass value="8.0"/>
+      <mass value="0.05"/>
       <origin xyz="0 0 0" rpy="0 0 0"/>
       <inertia
@@ -58,5 +58,5 @@
     <pose>0 0 0 0 0 0</pose>
     <inertial>
-      <mass value="8"/>
+      <mass value="0.05"/>
       <origin xyz="0 0 0" rpy="0 0 0"/>
       <inertia
@@ -79,5 +79,5 @@
     </visual>
   </link>
-  <link name='camera_pillar'>
+  <!-- <link name='camera_pillar'>
     <pose>0 0 0 0 0 0</pose>
     <inertial>
@@ -102,5 +102,5 @@
       </geometry>
     </visual>
-  </link>
+  </link>-->
   <joint type="continuous" name="left_wheel_hinge">
     <origin xyz="-0.107266 -0.242145 0.5" rpy=" 0 -1.5707 1.5707"/>
@@ -119,5 +119,5 @@
     <dynamics damping="1.0" friction="1.0"/>
   </joint>
-  <joint type="fixed" name="camera_pillar_hinge">
+  <!-- <joint type="fixed" name="camera_pillar_hinge">
     <origin xyz="-0.182538 0.002574 0.674205" rpy="-0.000428 0.002653 -0.024756"/>
     <child link="camera_pillar"/>
@@ -126,4 +126,4 @@
     <limit effort="10000" velocity="1000"/>
     <dynamics damping="1.0" friction="1.0"/>
-  </joint>
+  </joint>-->
 </robot>

Commit message: urdf made stable

File: robot/urdf/robot.xacro (robot description, xacro)
@@ -13,7 +13,7 @@
       <origin xyz="0 0 0.5" rpy=" 1.5707 0 1.5707"/>
       <inertia
-          ixx="1e-6" ixy="0" ixz="0"
-          iyy="1e-6" iyz="0"
-          izz="1e-6"
+          ixx="0.4298" ixy="0" ixz="0"
+          iyy="0.207" iyz="0"
+          izz="0.236"
       />
     </inertial>
@@ -21,5 +21,6 @@
       <origin xyz="0 0 0.5" rpy=" 1.5707 0 1.5707"/>
       <geometry>
-        <box size="0.1 0.1 0.1"/>
+        <!--<box size="1.0 1.0 1.0"/>-->
+        <mesh filename="package://robot/meshes/Dingo_without_tyre.dae"/>
       </geometry>
     </collision>
@@ -34,10 +35,10 @@
     <pose>0 0 0 0 0 0</pose>
     <inertial>
-      <mass value="0.05"/>
+      <mass value="0.35"/>
       <origin xyz="0 0 0" rpy="0 0 0"/>
       <inertia
-          ixx="0.1" ixy="0" ixz="0"
-          iyy="0.1" iyz="0"
-          izz="0.1"
+          ixx="0.000225" ixy="0" ixz="0"
+          iyy="0.000225" iyz="0"
+          izz="0.0004375"
       />
     </inertial>
@@ -58,10 +59,10 @@
     <pose>0 0 0 0 0 0</pose>
     <inertial>
-      <mass value="0.05"/>
+      <mass value="0.35"/>
       <origin xyz="0 0 0" rpy="0 0 0"/>
       <inertia
-          ixx="0.1" ixy="0" ixz="0"
-          iyy="0.1" iyz="0"
-          izz="0.1"
+          ixx="0.000225" ixy="0" ixz="0"
+          iyy="0.000225" iyz="0"
+          izz="0.0004375"
       />
     </inertial>

Commit message: camera added in the urdf

File: robot/urdf/robot.xacro (robot description, xacro)
@@ -80,5 +80,5 @@
     </visual>
   </link>
-  <!-- <link name='camera_pillar'>
+  <link name='camera_pillar'>
     <pose>0 0 0 0 0 0</pose>
     <inertial>
@@ -86,7 +86,7 @@
       <origin xyz="0 0 0" rpy="0 0 0"/>
       <inertia
-          ixx="0.1" ixy="0" ixz="0"
-          iyy="0.1" iyz="0"
-          izz="0.1"
+          ixx="0.0001979" ixy="0" ixz="0"
+          iyy="0.0001979" iyz="0"
+          izz="0.0000625"
       />
     </inertial>
@@ -94,5 +94,5 @@
       <origin xyz="0 0 0" rpy="0 0 0"/>
       <geometry>
-        <box size="0.05 0.05 0.2"/>
+        <cylinder radius="0.025" length="0.1"/>
       </geometry>
     </collision>
@@ -100,8 +100,32 @@
       <origin xyz="0 0 0" rpy="0 0 0"/>
       <geometry>
-        <box size="0.05 0.05 0.2"/>
+        <cylinder radius="0.025" length="0.1"/>
       </geometry>
     </visual>
-  </link>-->
+  </link>
+  <link name='camera_link'>
+    <pose>0 0 0 0 0 0</pose>
+    <inertial>
+      <mass value="0.2"/>
+      <origin xyz="0 0 0" rpy="0 0 0"/>
+      <inertia
+          ixx="0.0001979" ixy="0" ixz="0"
+          iyy="0.0001979" iyz="0"
+          izz="0.0000625"
+      />
+    </inertial>
+    <collision name='camera_link_collision'>
+      <origin xyz="0 0 0" rpy="0 0 0"/>
+      <geometry>
+        <mesh filename="package://robot/meshes/intel_realsense_camera.dae"/>
+      </geometry>
+    </collision>
+    <visual name='camera_link_visual'>
+      <origin xyz="0 0 0" rpy="0 0 0"/>
+      <geometry>
+        <mesh filename="package://robot/meshes/intel_realsense_camera.dae"/>
+      </geometry>
+    </visual>
+  </link>
   <joint type="continuous" name="left_wheel_hinge">
     <origin xyz="-0.107266 -0.242145 0.5" rpy=" 0 -1.5707 1.5707"/>
@@ -120,6 +144,6 @@
     <dynamics damping="1.0" friction="1.0"/>
   </joint>
-  <!-- <joint type="fixed" name="camera_pillar_hinge">
-    <origin xyz="-0.182538 0.002574 0.674205" rpy="-0.000428 0.002653 -0.024756"/>
+  <joint type="fixed" name="camera_pillar_hinge">
+    <origin xyz="-0.194581 0.000743 0.612654" rpy="-0.002050 -0.088042 -0.023313"/>
     <child link="camera_pillar"/>
     <parent link="robot_body"/>
@@ -127,4 +151,12 @@
     <limit effort="10000" velocity="1000"/>
     <dynamics damping="1.0" friction="1.0"/>
-  </joint>-->
+  </joint>
+  <joint type="fixed" name="camera_link_hinge">
+    <origin xyz="-0.020635 0.006883 0.064051" rpy="-1.57 0 1.57"/>
+    <child link="camera_link"/>
+    <parent link="camera_pillar"/>
+    <axis xyz="0 0 -1" rpy="0 0 0"/>
+    <limit effort="10000" velocity="1000"/>
+    <dynamics damping="1.0" friction="1.0"/>
+  </joint>
 </robot>

Commit message: colous added to urdf for gazebo

File: robot/urdf/robot.xacro (robot description, xacro)
@@ -160,3 +160,12 @@
     <dynamics damping="1.0" friction="1.0"/>
   </joint>
+  <gazebo reference="left_wheel">
+    <material>Gazebo/Black</material>
+  </gazebo>
+  <gazebo reference="right_wheel">
+    <material>Gazebo/Black</material>
+  </gazebo>
+  <gazebo reference="camera_pillar">
+    <material>Gazebo/Red</material>
+  </gazebo>
 </robot>

Commit message: urdf almost fine

File: robot/urdf/robot.xacro (robot description, xacro)
@@ -1,4 +1,7 @@
 <?xml version='1.0'?>
 <robot name="name" xmlns:xacro="http://www.ros.org/wiki/xacro">
+  <material name="black">
+    <color rgba="0 0 0 1"/>
+  </material>
   <link name='robot_footprint'> </link>
   <joint name="robot_footprint_joint" type="fixed">
@@ -11,5 +14,5 @@
     <inertial>
       <mass value="9"/>
-      <origin xyz="0 0 0.5" rpy=" 1.5707 0 1.5707"/>
+      <origin xyz="0 0 0" rpy=" 1.5707 0 1.5707"/>
       <inertia
           ixx="0.4298" ixy="0" ixz="0"
@@ -19,14 +22,14 @@
     </inertial>
     <collision name='robot_collision'>
-      <origin xyz="0 0 0.5" rpy=" 1.5707 0 1.5707"/>
+      <origin xyz="0 0 0" rpy=" 1.5707 0 1.5707"/>
       <geometry>
         <!--<box size="1.0 1.0 1.0"/>-->
-        <mesh filename="package://robot/meshes/Dingo_without_tyre.dae"/>
+        <mesh filename="package://robot/meshes/dingo_for_omni.dae"/>
       </geometry>
     </collision>
     <visual name='robot_visual'>
-      <origin xyz="0 0 0.5" rpy=" 1.5707 0 1.5707"/>
+      <origin xyz="0 0 0" rpy=" 1.5707 0 1.5707"/>
       <geometry>
-        <mesh filename="package://robot/meshes/Dingo_without_tyre.dae"/>
+        <mesh filename="package://robot/meshes/dingo_for_omni.dae"/>
       </geometry>
     </visual>
@@ -54,4 +57,5 @@
         <cylinder radius="0.05" length="0.015"/>
       </geometry>
+      <material name="black"/>
     </visual>
   </link>
@@ -78,28 +82,30 @@
         <cylinder radius="0.05" length="0.015"/>
       </geometry>
+      <material name="black"/>
     </visual>
   </link>
-  <link name='camera_pillar'>
+  <link name='omni_wheel'>
     <pose>0 0 0 0 0 0</pose>
     <inertial>
-      <mass value="0.2"/>
+      <mass value="0.35"/>
       <origin xyz="0 0 0" rpy="0 0 0"/>
       <inertia
-          ixx="0.0001979" ixy="0" ixz="0"
-          iyy="0.0001979" iyz="0"
-          izz="0.0000625"
+          ixx="0.0056" ixy="0" ixz="0"
+          iyy="0.0056" iyz="0"
+          izz="0.0056"
       />
     </inertial>
-    <collision name='pillar_collision'>
+    <collision name='omni_wheel_collision'>
       <origin xyz="0 0 0" rpy="0 0 0"/>
       <geometry>
-        <cylinder radius="0.025" length="0.1"/>
+        <sphere radius="0.02"/>
       </geometry>
     </collision>
-    <visual name='pillar_visual'>
+    <visual name='omni_wheel_visual'>
       <origin xyz="0 0 0" rpy="0 0 0"/>
       <geometry>
-        <cylinder radius="0.025" length="0.1"/>
+        <sphere radius="0.02"/>
       </geometry>
+      <material name="black"/>
     </visual>
   </link>
@@ -129,32 +135,32 @@
   </link>
   <joint type="continuous" name="left_wheel_hinge">
-    <origin xyz="-0.107266 -0.242145 0.5" rpy=" 0 -1.5707 1.5707"/>
+    <origin xyz="-0.100266 -0.242145 0.03" rpy=" 0 -1.5707 1.5707"/>
     <child link="left_wheel"/>
     <parent link="robot_body"/>
-    <axis xyz="0 0 1" rpy="0 0 0"/>
+    <axis xyz="0 1 0" rpy="0 0 0"/>
     <limit effort="10000" velocity="1000"/>
     <dynamics damping="1.0" friction="1.0"/>
   </joint>
   <joint type="continuous" name="right_wheel_hinge">
-    <origin xyz="-0.107266 0.242145 0.5" rpy=" 0 -1.5707 1.5707"/>
+    <origin xyz="-0.100266 0.242145 0.03" rpy=" 0 -1.5707 1.5707"/>
     <child link="right_wheel"/>
     <parent link="robot_body"/>
-    <axis xyz="0 0 1" rpy="0 0 0"/>
-    <limit effort="10000" velocity="1000"/>
-    <dynamics damping="1.0" friction="1.0"/>
-  </joint>
-  <joint type="fixed" name="camera_pillar_hinge">
-    <origin xyz="-0.194581 0.000743 0.612654" rpy="-0.002050 -0.088042 -0.023313"/>
-    <child link="camera_pillar"/>
-    <parent link="robot_body"/>
-    <axis xyz="0 0 1" rpy="0 0 0"/>
+    <axis xyz="0 1 0" rpy="0 0 0"/>
     <limit effort="10000" velocity="1000"/>
     <dynamics damping="1.0" friction="1.0"/>
   </joint>
   <joint type="fixed" name="camera_link_hinge">
-    <origin xyz="-0.020635 0.006883 0.064051" rpy="-1.57 0 1.57"/>
+    <origin xyz="-0.300635 0.0 0.05051" rpy="-1.57 0 1.57"/>
     <child link="camera_link"/>
-    <parent link="camera_pillar"/>
+    <parent link="robot_body"/>
     <axis xyz="0 0 -1" rpy="0 0 0"/>
+    <limit effort="10000" velocity="1000"/>
+    <dynamics damping="1.0" friction="1.0"/>
+  </joint>
+  <joint type="continuous" name="omni_wheel_hinge">
+    <origin xyz="0.233497 -0.000865 0" rpy="0.000212 -0.118296 -0.001802"/>
+    <child link="omni_wheel"/>
+    <parent link="robot_body"/>
+    <axis xyz="0 0 1" rpy="0 0 0"/>
     <limit effort="10000" velocity="1000"/>
     <dynamics damping="1.0" friction="1.0"/>
@@ -166,6 +172,6 @@
     <material>Gazebo/Black</material>
   </gazebo>
-  <gazebo reference="camera_pillar">
-    <material>Gazebo/Red</material>
+  <gazebo reference="omni_wheel">
+    <material>Gazebo/Black</material>
   </gazebo>
 </robot>

Commit message: Urdf updated

File: robot/urdf/robot.xacro (robot description, xacro)
@@ -1,4 +1,5 @@
 <?xml version='1.0'?>
 <robot name="name" xmlns:xacro="http://www.ros.org/wiki/xacro">
+  <xacro:include filename="$(find robot)/urdf/robot.gazebo" />
   <material name="black">
     <color rgba="0 0 0 1"/>
@@ -138,5 +139,5 @@
     <child link="left_wheel"/>
     <parent link="robot_body"/>
-    <axis xyz="0 1 0" rpy="0 0 0"/>
+    <axis xyz="0 0 1" rpy="0 0 0"/>
     <limit effort="10000" velocity="1000"/>
     <dynamics damping="1.0" friction="1.0"/>
@@ -146,5 +147,5 @@
     <child link="right_wheel"/>
     <parent link="robot_body"/>
-    <axis xyz="0 1 0" rpy="0 0 0"/>
+    <axis xyz="0 0 1" rpy="0 0 0"/>
     <limit effort="10000" velocity="1000"/>
     <dynamics damping="1.0" friction="1.0"/>
@@ -154,5 +155,5 @@
     <child link="camera_link"/>
     <parent link="robot_body"/>
-    <axis xyz="0 0 -1" rpy="0 0 0"/>
+    <axis xyz="0 0 1" rpy="0 0 0"/>
     <limit effort="10000" velocity="1000"/>
     <dynamics damping="1.0" friction="1.0"/>

Commit message: urdf updated

File: robot/urdf/robot.xacro (robot description, xacro)
@@ -1,4 +1,4 @@
 <?xml version='1.0'?>
-<robot name="name" xmlns:xacro="http://www.ros.org/wiki/xacro">
+<robot name="robot" xmlns:xacro="http://www.ros.org/wiki/xacro">
   <xacro:include filename="$(find robot)/urdf/robot.gazebo" />
   <material name="black">
@@ -117,7 +117,7 @@
       <origin xyz="0 0 0" rpy="0 0 0"/>
       <inertia
-          ixx="0.0001979" ixy="0" ixz="0"
-          iyy="0.0001979" iyz="0"
-          izz="0.0000625"
+          ixx="0.000196" ixy="0" ixz="0"
+          iyy="0.0000125875" iyz="0"
+          izz="0.0002044"
       />
     </inertial>
@@ -125,5 +125,5 @@
       <origin xyz="0 0 0" rpy="0 0 0"/>
       <geometry>
-        <mesh filename="package://robot/meshes/intel_realsense_camera.dae"/>
+        <mesh filename="package://robot/meshes/tracking_camera.dae"/>
       </geometry>
     </collision>
@@ -131,5 +131,5 @@
       <origin xyz="0 0 0" rpy="0 0 0"/>
       <geometry>
-        <mesh filename="package://robot/meshes/intel_realsense_camera.dae"/>
+        <mesh filename="package://robot/meshes/tracking_camera.dae"/>
       </geometry>
     </visual>

Commit message: urdf - joint of camera updated

File: robot/urdf/robot.xacro (robot description, xacro)
@@ -152,5 +152,5 @@
   </joint>
   <joint type="fixed" name="camera_link_hinge">
-    <origin xyz="-0.300635 0.0 0.05051" rpy="-1.57 0 1.57"/>
+    <origin xyz="-0.285635 0.0 0.05051" rpy="-1.57 0 1.57"/>
     <child link="camera_link"/>
     <parent link="robot_body"/>
